File: pcb/flicker-light-node-hardware.kicad_pcb (KiCad board)
At the start: 2 copper layers, 0 parts

Commit message: Finished up first draft of schematic, finding all parts, debating switch, or if I should just make users disconnect battery, I know the right answer, but only have so much space... I am thinking to moving to a smaller connector. Started PCB layout, using the following box http://www.budind.com/pdf/hb3660.pdf
Parts:
- added C1: 4.7uF, Capacitors_SMD:C_0805, F.Cu at (262.5, 162.3)
- added C2: .1uF, Capacitors_SMD:C_0603, F.Cu at (254.6, 146.7)
- added C3: .1uF, Capacitors_SMD:C_0603, F.Cu at (271.8, 127.0)
- added C4: 4.7uF, Capacitors_SMD:C_0805, F.Cu at (241.3, 176.5)
- added C5: 4.7uF, Capacitors_SMD:C_0805, F.Cu at (237.5, 170.2)
- added C6: .1uF, Capacitors_SMD:C_0603, F.Cu at (284.6, 149.2)
- added C7: .1uF, Capacitors_SMD:C_0603, F.Cu at (287.1, 158.1)
- added D1: GREEN, LEDs:LED_0603, F.Cu at (287.1, 146.7)
- added F1: PTC RESTTBLE 2.6A 16V CHIP 1812, Resistors_SMD:R_1812, F.Cu at (188.0, 125.7)
- added IC1: ATMEGA168PA-MM, Housings_DFN_QFN:QFN-28-1EP_4x4mm_Pitch0.4mm, F.Cu at (222.2, 132.1)
- added P1: CONN_01X06, xess:HDR_1x6, F.Cu at (234.9, 130.8)
- added P2: CONN_01X02, xess:HDR_1x2, F.Cu at (181.6, 124.5)
- added P3: CONN_02X04, Radio_Modules:NRF24L01, F.Cu at (199.4, 141.0)
- added P4: CONN_02X03, xess:HDR_2x3, F.Cu at (233.7, 143.5)
- added P5: CONN_01X04, Connectors_Molex:Molex_Microfit3_Header_02x02_Straight_43045-0428, F.Cu at (203.2, 113.0)
- added P6: CONN_01X04, Connectors_Molex:Molex_Microfit3_Header_02x02_Straight_43045-0428, F.Cu at (215.9, 113.0)
- added Q1: BSS138, TO_SOT_Packages_SMD:SOT-23, F.Cu at (280.8, 151.8)
- added Q2: BSS138, TO_SOT_Packages_SMD:SOT-23, F.Cu at (291.0, 156.8)
- added Q3: BSS138, TO_SOT_Packages_SMD:SOT-23, F.Cu at (296.0, 156.8)
- added Q4: BSS138, TO_SOT_Packages_SMD:SOT-23, F.Cu at (262.4, 156.1)
- added Q5: BSS138, TO_SOT_Packages_SMD:SOT-23, F.Cu at (267.6, 163.6)
- added Q6: BSS138, TO_SOT_Packages_SMD:SOT-23, F.Cu at (280.8, 144.1)
- added R1: 200K, Resistors_SMD:R_0603, F.Cu at (298.6, 156.8)
- added R2: 100K, Resistors_SMD:R_0603, F.Cu at (291.0, 142.9)
- added R3: 10K, Resistors_SMD:R_0603, F.Cu at (288.4, 151.8)
- added R4: 1K, Resistors_SMD:R_0603, F.Cu at (287.1, 144.1)
- added REF**: MountingHole_3.5mm_Pad, Mounting_Holes:MountingHole_3.5mm_Pad, F.Cu at (193.7, 118.1)
- added REF**: MountingHole_3.5mm_Pad, Mounting_Holes:MountingHole_3.5mm_Pad, F.Cu at (221.6, 119.1)
- added REF**: MountingHole_3.5mm_Pad, Mounting_Holes:MountingHole_3.5mm_Pad, F.Cu at (193.7, 146.2)
- added REF**: MountingHole_3.5mm_Pad, Mounting_Holes:MountingHole_3.5mm_Pad, F.Cu at (221.6, 146.2)
- added U2: LD1117S33CTR, TO_SOT_Packages_SMD:SOT-223, F.Cu at (243.8, 171.4)
Other:
- board outline added: 59.7 x 48.3 mm
